File: ESP32 Drone Section_2/ESP32-drone-project 1.00.kicad_pcb (KiCad board)
At the start: 2 copper layers, 62 parts, among them Q1 DMG2302U, Q2 DMG2302U, Q3 DMG2302U, Q4 DMG2302U, U1 ESP32-C6-MINI-1, U2 BMI088, U3 BMP280, U4 VL53L1CXV0FY1, U5 XC6220B331MR, U6 XC6220B331MR, U7 XC6220B331MR

Commit message: Add files via upload
Parts:
- removed TP38, TP39, TP43, TP44: TestPoint, TestPoint:TestPoint_Pad_D1.0mm
- moved TP42 76.3 mm to (35.2, 19.8)
- moved TP41 73.4 mm to (59.2, 15.2)
- moved TP40 72.2 mm to (63.5, 15.5)
- moved TP45 40.6 mm to (35.0, 15.8)
- moved TP24 40.2 mm to (50.8, 47.5)
- moved TP26 36.0 mm to (50.5, 44.5)
- moved TP37 30.9 mm to (43.0, 56.0)
- moved TP23 30.3 mm to (58.2, 81.2)
- moved TP28 28.2 mm to (50.5, 41.8)
- moved TP25 25.5 mm to (37.5, 44.2)
- moved TP27 24.3 mm to (37.5, 47.2)
- moved TP46 20.4 mm to (53.2, 29.0)
- moved Q4 9.41 mm to (35.8, 29.0)
- moved D5 0.25 mm to (45.8, 78.8)
Connections:
- U1 pad 17: Net-(U1-IO12) -> unconnected-(U1-IO12-Pad17)
- U1 pad 24: Net-(U1-IO18) -> unconnected-(U1-IO18-Pad24)
- U1 pad 27: Net-(Q2-G) -> Net-(Q4-G)
- U1 pad 28: Net-(Q4-G) -> Net-(Q2-G)
- U1 pad 6: Net-(U1-IO3) -> unconnected-(U1-IO3-Pad6)
- U1 pad 9: Net-(U1-IO4) -> unconnected-(U1-IO4-Pad9)
Routing:
- net Net-(BT1-+): track 0.00 -> 426.0 mm, vias 0 -> 1
- net Net-(D5-DIN): track 0.00 -> 83.4 mm
- net Net-(Q2-G): track 0.00 -> 74.2 mm
- net Net-(U1-IO2): track 0.00 -> 64.8 mm, vias 0 -> 1
- net Net-(U1-IO8): track 0.00 -> 57.5 mm, vias 0 -> 2
- net Net-(Q4-G): track 0.00 -> 55.4 mm, vias 0 -> 2
- net Net-(D5-DOUT): track 0.00 -> 38.4 mm
- net Net-(Q1-G): track 0.00 -> 34.8 mm
- net Net-(U2-INT1): track 0.00 -> 26.3 mm
- net Net-(D3-A): track 0.00 -> 25.8 mm
- net Net-(D2-K): track 0.00 -> 20.3 mm
- net Net-(D4-A): track 0.00 -> 20.0 mm
- net Net-(D2-A): track 0.00 -> 17.8 mm
- net Net-(D1-A): track 0.00 -> 17.4 mm
- net Net-(U1-IO0): track 0.00 -> 13.7 mm
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