File: ESP32 Drone Section_2/ESP32-drone-project 1.00.kicad_sch (KiCad schematic)
At the start: 64 parts, among them Q1 DMG2302U, Q2 DMG2302U, Q3 DMG2302U, Q4 DMG2302U, U1 ESP32-C6-MINI-1, U2 BMI088, U3 BMP280, U4 VL53L1CXV0FY1, U5 XC6220B331MR, U6 XC6220B331MR, U7 XC6220B331MR

Commit message: Add files via upload
Parts:
- removed TP38, TP39, TP43, TP44: TestPoint, TestPoint:TestPoint_Pad_D1.0mm, symbol Connector:TestPoint
Connections:
- net at Q2.1 (G): now also U1.28 (IO22); no longer U1.27 (IO21)
- net at Q4.1 (G): now also U1.27 (IO21); no longer U1.28 (IO22)
